Commit message: param tuning

File: urdf/udacity_bot.xacro (robot description, xacro)
@@ -70,5 +70,5 @@
   <link name='left_wheel'>
     <inertial>
-      <mass value="3.0"/>
+      <mass value="10.0"/>
       <origin xyz="0.0 0 0" rpy=" 0 1.5707 1.5707"/>
       <inertia
@@ -93,5 +93,5 @@
   <link name='right_wheel'>
     <inertial>
-      <mass value="3.0"/>
+      <mass value="10.0"/>
       <origin xyz="0.0 0 0" rpy=" 0 1.5707 1.5707"/>
       <inertia
