Commit message: coloring material

File: urdf/robond_bot.xacro (robot description, xacro)
@@ -54,4 +54,7 @@
         <sphere radius="0.1"/>
       </geometry>
+       <material name="Cyan">
+          <color rgba="0 1.0 1.0 1.0"/>
+        </material>
     </visual>
     <collision name='front_caster_collision'>
